File: 8SiPMAdaptorBoard/AdaptorBoard/AdaptorBoard.kicad_sch (KiCad schematic)
At the start: 17 parts, among them J1 FFC_Connector_Vertical, J10 Signal1, J11 Signal2, J12 Signal3, J13 Signal4, J14 Signal8, J15 Signal7, J16 Signal6, J17 Signal5, J2 FFC_Connector_Vertical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

Commit message: Update SiPM_Adaptor_Design
Parts:
- removed J11: Signal2, Connector_Coaxial:BNC_PanelMountable_Vertical, symbol BNC5-J-P-GN-ST-TH2D:BNC5-J-P-GN-ST-TH2D
- removed J12: Signal3, Connector_Coaxial:BNC_PanelMountable_Vertical, symbol BNC5-J-P-GN-ST-TH2D:BNC5-J-P-GN-ST-TH2D
- removed J13: Signal4, Connector_Coaxial:BNC_PanelMountable_Vertical, symbol BNC5-J-P-GN-ST-TH2D:BNC5-J-P-GN-ST-TH2D
- removed J14: Signal8, Connector_Coaxial:BNC_PanelMountable_Vertical, symbol BNC5-J-P-GN-ST-TH2D:BNC5-J-P-GN-ST-TH2D
- removed J15: Signal7, Connector_Coaxial:BNC_PanelMountable_Vertical, symbol BNC5-J-P-GN-ST-TH2D:BNC5-J-P-GN-ST-TH2D
- removed J16: Signal6, Connector_Coaxial:BNC_PanelMountable_Vertical, symbol BNC5-J-P-GN-ST-TH2D:BNC5-J-P-GN-ST-TH2D
- removed J17: Signal5, Connector_Coaxial:BNC_PanelMountable_Vertical, symbol BNC5-J-P-GN-ST-TH2D:BNC5-J-P-GN-ST-TH2D
- removed J2, J3, J4, J5, J6, J7, J8: FFC_Connector_Vertical, symbol FFCZF5S-10-03-T-WT:ZF5S-10-03-T-WT
- removed J9: Conn_01x05_Pin, symbol Connector:Conn_01x05_Pin
- added +2V5, -2V5, GND1, SiPM_Bias1: Conn_01x09, Connector_PinHeader_1.00mm:PinHeader_1x09_P1.00mm_Vertical, symbol Connector_Generic:Conn_01x09
- added BNC1: Signal1, BNC5-J-P-GN-ST-TH2D:SAMTEC_BNC5-J-P-GN-ST-TH2D, symbol BNC5-J-P-GN-ST-TH2D:BNC5-J-P-GN-ST-TH2D
- added BNC2: Signal2, BNC5-J-P-GN-ST-TH2D:SAMTEC_BNC5-J-P-GN-ST-TH2D, symbol BNC5-J-P-GN-ST-TH2D:BNC5-J-P-GN-ST-TH2D
- added BNC3: Signal3, BNC5-J-P-GN-ST-TH2D:SAMTEC_BNC5-J-P-GN-ST-TH2D, symbol BNC5-J-P-GN-ST-TH2D:BNC5-J-P-GN-ST-TH2D
- added BNC5: Signal5, BNC5-J-P-GN-ST-TH2D:SAMTEC_BNC5-J-P-GN-ST-TH2D, symbol BNC5-J-P-GN-ST-TH2D:BNC5-J-P-GN-ST-TH2D
- added BNC6: Signal6, BNC5-J-P-GN-ST-TH2D:SAMTEC_BNC5-J-P-GN-ST-TH2D, symbol BNC5-J-P-GN-ST-TH2D:BNC5-J-P-GN-ST-TH2D
- added BNC7: Signal7, BNC5-J-P-GN-ST-TH2D:SAMTEC_BNC5-J-P-GN-ST-TH2D, symbol BNC5-J-P-GN-ST-TH2D:BNC5-J-P-GN-ST-TH2D
- added BNC8: Signal8, BNC5-J-P-GN-ST-TH2D:SAMTEC_BNC5-J-P-GN-ST-TH2D, symbol BNC5-J-P-GN-ST-TH2D:BNC5-J-P-GN-ST-TH2D
- added FFC1, FFC2, FFC3, FFC5, FFC6, FFC7, FFC8: FFC_Connector_Vertical, FFC_10position_vertical:SAMTEC_ZF5S-10-03-T-WT, symbol FFCZF5S-10-03-T-WT:ZF5S-10-03-T-WT
- added PIN1, PIN2, PIN3, PIN4, PIN5, PIN6, PIN7, PIN8: Conn_01x04_Pin, Connector_PinHeader_1.00mm:PinHeader_1x04_P1.00mm_Vertical, symbol Connector:Conn_01x04_Pin
- BNC4: renamed from J10; value Signal1 -> Signal4; footprint Connector_Coaxial:BNC_PanelMountable_Vertical -> BNC5-J-P-GN-ST-TH2D:SAMTEC_BNC5-J-P-GN-ST-TH2D
- FFC4: renamed from J1; footprint (none) -> FFC_10position_vertical:SAMTEC_ZF5S-10-03-T-WT
Connections:
- net at BNC4.S_1, BNC4.S_2, BNC4.S_3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: now also FFC4.03 (Earth), FFC4.05 (Earth), FFC4.06 (Earth), FFC4.10 (Earth), PIN4.1 (Pin_1)
- net at FFC4.07 (-2V5): now also PIN4.2 (Pin_2)
- net at FFC4.08 (+2V5): now also PIN4.3 (Pin_3)
- net at FFC4.09 (V_Bias): now also PIN4.4 (Pin_4)
- new net: BNC2.S_1, BNC2.S_2, BNC2.S_3, FFC2.01 (Earth), FFC2.03 (Earth), FFC2.05 (Earth), FFC2.06 (Earth), FFC2.10 (Earth), PIN2.1 (Pin_1)
- new net: FFC2.07 (-2V5), PIN2.2 (Pin_2)
- new net: FFC2.08 (+2V5), PIN2.3 (Pin_3)
- new net: FFC2.09 (V_Bias), PIN2.4 (Pin_4)
- new net: BNC8.1, FFC8.02 (Signal)
- new net: BNC8.S_1, BNC8.S_2, BNC8.S_3, FFC8.01 (Earth), FFC8.03 (Earth), FFC8.05 (Earth), FFC8.06 (Earth), FFC8.10 (Earth), PIN8.1 (Pin_1)
- new net: FFC8.07 (-2V5), PIN8.2 (Pin_2)
- new net: FFC8.08 (+2V5), PIN8.3 (Pin_3)
- new net: FFC8.09 (V_Bias), PIN8.4 (Pin_4)
- new net: BNC1.S_1, BNC1.S_2, BNC1.S_3, FFC1.01 (Earth), FFC1.03 (Earth), FFC1.05 (Earth), FFC1.06 (Earth), FFC1.10 (Earth), PIN1.1 (Pin_1)
- new net: BNC1.1, FFC1.02 (Signal)
- new net: FFC1.07 (-2V5), PIN1.2 (Pin_2)
- new net: FFC1.08 (+2V5), PIN1.3 (Pin_3)
- new net: FFC1.09 (V_Bias), PIN1.4 (Pin_4)
- new net: BNC5.S_1, BNC5.S_2, BNC5.S_3, FFC5.01 (Earth), FFC5.03 (Earth), FFC5.05 (Earth), FFC5.06 (Earth), FFC5.10 (Earth), PIN5.1 (Pin_1)
- new net: BNC5.1, FFC5.02 (Signal)
- new net: FFC5.07 (-2V5), PIN5.2 (Pin_2)
- new net: FFC5.08 (+2V5), PIN5.3 (Pin_3)
- new net: FFC5.09 (V_Bias), PIN5.4 (Pin_4)
- new net: BNC3.1, FFC3.02 (Signal)
- new net: BNC3.S_1, BNC3.S_2, BNC3.S_3, FFC3.01 (Earth), FFC3.03 (Earth), FFC3.05 (Earth), FFC3.06 (Earth), FFC3.10 (Earth), PIN3.1 (Pin_1)
- new net: BNC2.1, FFC2.02 (Signal)
- new net: BNC7.S_1, BNC7.S_2, BNC7.S_3, FFC7.01 (Earth), FFC7.03 (Earth), FFC7.05 (Earth), FFC7.06 (Earth), FFC7.10 (Earth), PIN7.1 (Pin_1)
- new net: BNC7.1, FFC7.02 (Signal)
- new net: FFC7.07 (-2V5), PIN7.2 (Pin_2)
- new net: FFC7.08 (+2V5), PIN7.3 (Pin_3)
- new net: FFC7.09 (V_Bias), PIN7.4 (Pin_4)
- new net: BNC6.1, FFC6.02 (Signal)
- new net: BNC6.S_1, BNC6.S_2, BNC6.S_3, FFC6.01 (Earth), FFC6.03 (Earth), FFC6.05 (Earth), FFC6.06 (Earth), FFC6.10 (Earth), PIN6.1 (Pin_1)
- new net: FFC6.07 (-2V5), PIN6.2 (Pin_2)
- new net: FFC6.08 (+2V5), PIN6.3 (Pin_3)
- new net: FFC6.09 (V_Bias), PIN6.4 (Pin_4)
- new net: FFC3.07 (-2V5), PIN3.2 (Pin_2)
- new net: FFC3.08 (+2V5), PIN3.3 (Pin_3)
- new net: FFC3.09 (V_Bias), PIN3.4 (Pin_4)
Other:
- company: (none) -> HKUST
- title: (none) -> PCB_SiPMAdaptorToBNC
- moved on the sheet: BNC4, FFC4
