File: 8SiPMAdaptorBoard/AdaptorBoard/AdaptorBoard.kicad_pcb (KiCad board)
At the start: 2 copper layers, 86 x 63 mm, 28 parts

Commit message: Update SiPM_Adaptor_Design
Routing:
- net Net-(FFC8-Signal): track 0.00 -> 14.4 mm
- net Net-(FFC7-Signal): track 0.00 -> 14.3 mm
Changed lines of the file:
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@@
 	(gr_text "GND\n-2V5\n+2V5\nV_Bias"
 		(at 71 43 0)
-		(layer "Edge.Cuts")
+		(layer "Edge.Cuts" knockout)
 		(effects
 			(font
@@
 	)
 	(segment
+		(start 93.5 53.183514)
+		(end 90.768986 50.4525)
+		(width 0.2)
+		(layer "F.Cu")
+		(net 14)
+	)
+	(segment
+		(start 90.768986 50.4525)
+		(end 87.5075 50.4525)
+		(width 0.2)
+		(layer "F.Cu")
+		(net 14)
+	)
+	(segment
+		(start 87.5075 50.4525)
+		(end 84.14 53.82)
+		(width 0.2)
+		(layer "F.Cu")
+		(net 14)
+	)
+	(segment
+		(start 93.5 55.57)
+		(end 93.5 53.183514)
+		(width 0.2)
+		(layer "F.Cu")
+		(net 14)
+	)
+	(segment
+		(start 87.575 36.745)
+		(end 84 40.32)
+		(width 0.2)
+		(layer "F.Cu")
+		(net 15)
+	)
+	(segment
+		(start 93.36 42.07)
+		(end 93.36 39.683514)
+		(width 0.2)
+		(layer "F.Cu")
+		(net 15)
+	)
+	(segment
+		(start 93.36 39.683514)
+		(end 90.421486 36.745)
+		(width 0.2)
+		(layer "F.Cu")
+		(net 15)
+	)
+	(segment
+		(start 90.421486 36.745)
+		(end 87.575 36.745)
+		(width 0.2)
+		(layer "F.Cu")
+		(net 15)
+	)
+	(segment

Commit message: Update on the PCB board
Routing:
- net Net-(FFC7-+2V5): track 0.00 -> 6.38 mm
- net Net-(FFC6-Signal): track 14.3 -> 19.2 mm
- net Net-(FFC7-Signal): track 14.3 -> 19.2 mm
- net Net-(FFC8-Signal): track 14.4 -> 19.2 mm
- net Net-(FFC7--2V5): track 0.00 -> 4.45 mm
- net Net-(FFC5-Signal): track 15.1 -> 19.2 mm
- net Net-(FFC7-V_Bias): track 0.00 -> 4.03 mm
- net Net-(FFC2-Signal): track 17.4 -> 21.4 mm
- net Net-(FFC3-Signal): track 17.6 -> 21.4 mm
- net Net-(FFC1-Signal): track 18.1 -> 21.6 mm
- net Net-(FFC4-Signal): track 18.1 -> 21.1 mm

Commit message: More update on adaptor board
Parts:
- moved V_Bias1 38.5 mm to (71.0, 89.2)
- moved GND1 38.3 mm to (71.0, 76.0)
- moved -2V5 38.2 mm to (71.0, 63.2)
- moved +2V5 38.1 mm to (71.0, 49.0)
- renumbered SiPM_Bias1 to V_Bias1
Other:
- board size 86 x 63 mm -> 58.8 x 63 mm
- board text added: "Orientation"
Changed lines of the file:
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@@
 	(footprint "Connector_PinHeader_1.00mm:PinHeader_1x09_P1.00mm_Vertical"
 		(layer "F.Cu")
-		(at 109 71 90)
+		(at 71 76 90)
 		(descr "Through hole straight pin header, 1x09, 1.00mm pitch, single row")
 		(tags "Through hole pin header THT 1x09 1.00mm single row")
@@
 	(footprint "Connector_PinHeader_1.00mm:PinHeader_1x09_P1.00mm_Vertical"
 		(layer "F.Cu")
-		(at 109 83 90)
+		(at 71 89.25 90)
 		(descr "Through hole straight pin header, 1x09, 1.00mm pitch, single row")
 		(tags "Through hole pin header THT 1x09 1.00mm single row")
-		(property "Reference" "SiPM_Bias1"
-			(at 0 -2 -90)
+		(property "Reference" "V_Bias1"
+			(at 0 -2 270)
 			(layer "F.SilkS")
 			(effects
@@
 	(footprint "Connector_PinHeader_1.00mm:PinHeader_1x09_P1.00mm_Vertical"
 		(layer "F.Cu")
-		(at 109 47 90)
+		(at 71 49 90)
 		(descr "Through hole straight pin header, 1x09, 1.00mm pitch, single row")
 		(tags "Through hole pin header THT 1x09 1.00mm single row")
@@
 	(footprint "Connector_PinHeader_1.00mm:PinHeader_1x09_P1.00mm_Vertical"
 		(layer "F.Cu")
-		(at 109 59 90)
+		(at 71 63.25 90)
 		(descr "Through hole straight pin header, 1x09, 1.00mm pitch, single row")
 		(tags "Through hole pin header THT 1x09 1.00mm single row")
@@
 	(gr_rect
 		(start 44 32)
-		(end 130 95)
+		(end 102.75 95)
 		(stroke
 			(width 0.05)
@@
 		(layer "Edge.Cuts")
 	)
+	(gr_text "Orientation"
+		(at 84 55.75 90)
+		(layer "F.SilkS")
+		(effects
+			(font
+				(size 1 1)
+				(thickness 0.1)
+			)
+			(justify bottom)
+		)
+	)
+	(gr_text "Orientation"
+		(at 84 82.25 90)
+		(layer "F.SilkS")
+		(effects
+			(font
+				(size 1 1)
+				(thickness 0.1)
+			)
+			(justify bottom)
+		)
+	)
 	(gr_text "GND\n-2V5\n+2V5\nV_Bias"
 		(at 75 83 0)
-		(layer "Edge.Cuts")
+		(layer "F.SilkS")
 		(effects
 			(font
@@
 	(gr_text "GND\n-2V5\n+2V5\nV_Bias"
 		(at 75 57 0)
-		(layer "Edge.Cuts")
+		(layer "F.SilkS")
 		(effects
 			(font
@@
 		)
 	)
+	(gr_text "Orientation"
+		(at 84 42.25 90)
+		(layer "F.SilkS")
+		(effects
+			(font
+				(size 1 1)
+				(thickness 0.1)
+			)
+			(justify bottom)
+		)
+	)
 	(gr_text "GND\n-2V5\n+2V5\nV_Bias"
 		(at 71 83 0)
-		(layer "Edge.Cuts")
+		(layer "F.SilkS")
 		(effects
 			(font
@@
 		)
 	)
+	(gr_text "Orientation"
+		(at 66 42.25 90)
+		(layer "F.SilkS")
+		(effects
+			(font
+				(size 1 1)
+				(thickness 0.1)
+			)
+			(justify bottom)
+		)
+	)
 	(gr_text "GND\n-2V5\n+2V5\nV_Bias"
 		(at 71 43 0)
-		(layer "Edge.Cuts")
+		(layer "F.SilkS")
 		(effects
 			(font
@@
 		)
 	)
+	(gr_text "Orientation"
+		(at 66.25 55.75 90)
+		(layer "F.SilkS")
+		(effects
+			(font
+				(size 1 1)
+				(thickness 0.1)
+			)
+			(justify bottom)
+		)
+	)
+	(gr_text "Orientation"
+		(at 66.25 69.25 90)
+		(layer "F.SilkS")
+		(effects
+			(font
+				(size 1 1)
+				(thickness 0.1)
+			)
+			(justify bottom)
+		)
+	)
 	(gr_text "GND\n-2V5\n+2V5\nV_Bias"
 		(at 71 70 0)
-		(layer "Edge.Cuts")
+		(layer "F.SilkS")
 		(effects
 			(font
@@
 	(gr_text "GND\n-2V5\n+2V5\nV_Bias"
 		(at 75 70 0)
-		(layer "Edge.Cuts")
+		(layer "F.SilkS")
 		(effects
 			(font
@@
 		)
 	)
+	(gr_text "Orientation"
+		(at 66.25 82.25 90)
+		(layer "F.SilkS")
+		(effects
+			(font
+				(size 1 1)
+				(thickness 0.1)
+			)
+			(justify bottom)
+		)
+	)
+	(gr_text "Orientation"
+		(at 84 69.25 90)
+		(layer "F.SilkS")
+		(effects
+			(font
+				(size 1 1)
+				(thickness 0.1)
+			)
+			(justify bottom)
+		)
+	)
 	(gr_text "GND\n-2V5\n+2V5\nV_Bias"
 		(at 71 57 0)
-		(layer "Edge.Cuts")
+		(layer "F.SilkS")
 		(effects
 			(font
@@
 	(gr_text "GND\n-2V5\n+2V5\nV_Bias"
 		(at 75 43 0)
-		(layer "Edge.Cuts")
+		(layer "F.SilkS")
 		(effects
 			(font

Commit message: More update on adaptor board
Other:
- board text added: "Solder all of the pins"
- board text added: "UST Phys SiPM adaptor board 2024 03 26 Eltis"
Changed lines of the file:
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@@
 		(tags "Through hole pin header THT 1x09 1.00mm single row")
 		(property "Reference" "V_Bias1"
-			(at 0 -2 270)
+			(at 0 -2 -90)
 			(layer "F.SilkS")
 			(effects
@@
 		(layer "Edge.Cuts")
 	)
+	(gr_text "Solder all of the pins"
+		(at 75 87.5 0)
+		(layer "B.SilkS")
+		(effects
+			(font
+				(size 1 1)
+				(thickness 0.1)
+			)
+			(justify bottom mirror)
+		)
+	)
+	(gr_text "Solder all of the pins"
+		(at 75 61.75 0)
+		(layer "B.SilkS")
+		(effects
+			(font
+				(size 1 1)
+				(thickness 0.1)
+			)
+			(justify bottom mirror)
+		)
+	)
+	(gr_text "UST Phys SiPM adaptor board\n2024 03 26\nEltis"
+		(at 67.5 94.25 0)
+		(layer "B.SilkS")
+		(effects
+			(font
+				(size 1 1)
+				(thickness 0.1)
+			)
+			(justify left bottom mirror)
+		)
+	)
+	(gr_text "Solder all of the pins"
+		(at 75 47.25 0)
+		(layer "B.SilkS")
+		(effects
+			(font
+				(size 1 1)
+				(thickness 0.1)
+			)
+			(justify bottom mirror)
+		)
+	)
+	(gr_text "Solder all of the pins"
+		(at 75 74.5 0)
+		(layer "B.SilkS")
+		(effects
+			(font
+				(size 1 1)
+				(thickness 0.1)
+			)
+			(justify bottom mirror)
+		)
+	)
 	(gr_text "Orientation"
