File: 8SiPMAdaptorBoard/LEMOAdaptorBoard4/LEMOAdaptorBoard4.kicad_sch (KiCad schematic)
At the start: 17 parts

Commit message: More LEMO adaptor design
Parts:
- FFC1, FFC2, FFC3, FFC4, FFC5, FFC6, FFC7, FFC8: footprint FFC_10position_vertical:SAMTEC_ZF5S-10-03-T-WT -> FFC_10position_connector:SAMTEC_ZF5S-10-01-T-WT
Changed lines of the file:
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@@
 			)
 		)
-		(property "Footprint" "FFC_10position_vertical:SAMTEC_ZF5S-10-03-T-WT"
+		(property "Footprint" "FFC_10position_connector:SAMTEC_ZF5S-10-01-T-WT"
 			(at 45.72 73.66 0)
 			(effects
@@
 			)
 		)
-		(property "Footprint" "FFC_10position_vertical:SAMTEC_ZF5S-10-03-T-WT"
+		(property "Footprint" "FFC_10position_connector:SAMTEC_ZF5S-10-01-T-WT"
 			(at 45.72 154.94 0)
 			(effects
@@
 			)
 		)
-		(property "Footprint" "FFC_10position_vertical:SAMTEC_ZF5S-10-03-T-WT"
+		(property "Footprint" "FFC_10position_connector:SAMTEC_ZF5S-10-01-T-WT"
 			(at 45.72 114.3 0)
 			(effects
@@
 			)
 		)
-		(property "Footprint" "FFC_10position_vertical:SAMTEC_ZF5S-10-03-T-WT"
+		(property "Footprint" "FFC_10position_connector:SAMTEC_ZF5S-10-01-T-WT"
 			(at 153.67 74.93 0)
 			(effects
@@
 			)
 		)
-		(property "Footprint" "FFC_10position_vertical:SAMTEC_ZF5S-10-03-T-WT"
+		(property "Footprint" "FFC_10position_connector:SAMTEC_ZF5S-10-01-T-WT"
 			(at 153.67 31.75 0)
 			(effects
@@
 			)
 		)
-		(property "Footprint" "FFC_10position_vertical:SAMTEC_ZF5S-10-03-T-WT"
+		(property "Footprint" "FFC_10position_connector:SAMTEC_ZF5S-10-01-T-WT"
 			(at 153.67 157.48 0)
 			(effects
@@
 			)
 		)
-		(property "Footprint" "FFC_10position_vertical:SAMTEC_ZF5S-10-03-T-WT"
+		(property "Footprint" "FFC_10position_connector:SAMTEC_ZF5S-10-01-T-WT"
 			(at 153.67 116.84 0)
 			(effects
@@
 			)
 		)
-		(property "Footprint" "FFC_10position_vertical:SAMTEC_ZF5S-10-03-T-WT"
+		(property "Footprint" "FFC_10position_connector:SAMTEC_ZF5S-10-01-T-WT"
 			(at 45.72 33.02 0)
 			(effects

Commit message: Update LEMOAdaptorBoard4 for horizontal FFC connector
Parts:
- added H1, H2, H3, H4: MountingHole, MountingHole:MountingHole_5mm, symbol Mechanical:MountingHole
- Power1: footprint Connector_PinHeader_1.00mm:PinHeader_1x04_P1.00mm_Vertical -> Connector:FanPinHeader_1x04_P2.54mm_Vertical

Commit message: Some more update
Parts:
- removed H1, H2, H3, H4: MountingHole, MountingHole:MountingHole_5mm, symbol Mechanical:MountingHole
- added H1, H2, H3, H4: MountingHole_Pad, MountingHole:MountingHole_5mm_Pad, symbol Mechanical:MountingHole_Pad
Changed lines of the file:
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@@
-	)
-	(symbol
-		(lib_id "Mechanical:MountingHole")
-		(at 207.0283 49.6787 0)
-		(unit 1)
-		(exclude_from_sim yes)
-		(in_bom no)
-		(on_board yes)
-		(dnp no)
-		(fields_autoplaced yes)
-		(property "Reference" "H4"
-			(at 209.5683 48.4086 0)
-			(effects
-				(font
-					(size 1.27 1.27)
-				)
-				(justify left)
-			)
-		)
-		(property "Value" "MountingHole"
-			(at 209.5683 50.9486 0)
-			(effects
-				(font
-					(size 1.27 1.27)
-				)
-				(justify left)
-			)
-		)
-		(property "Footprint" "MountingHole:MountingHole_5mm"
-			(at 207.0283 49.6787 0)
-			(effects
-				(font
-					(size 1.27 1.27)
-				)
-				(hide yes)
-			)
-		)
-		(property "Datasheet" "~"
-			(at 207.0283 49.6787 0)
-			(effects
-				(font
-					(size 1.27 1.27)
-				)
-				(hide yes)
-			)
-		)
-		(property "Description" "Mounting Hole without connection"
-			(at 207.0283 49.6787 0)
-			(effects
-				(font
-					(size 1.27 1.27)
-				)
-				(hide yes)
-			)
-		)
-		(instances
-			(project "LEMOAdaptorBoard4"
-				(path "/90a29a6b-0930-4b18-ad75-feedfe88ac78"
-					(reference "H4")
-					(unit 1)
-				)
-			)
-		)
 	)
 	(symbol
@@
 	)
 	(symbol
-		(lib_id "Mechanical:MountingHole")
-		(at 208.28 41.91 0)
-		(unit 1)
-		(exclude_from_sim yes)
-		(in_bom no)
-		(on_board yes)
-		(dnp no)
-		(fields_autoplaced yes)
-		(property "Reference" "H3"
-			(at 210.82 40.6399 0)
-			(effects
-				(font
-					(size 1.27 1.27)
-				)
-				(justify left)
-			)
-		)
-		(property "Value" "MountingHole"
-			(at 210.82 43.1799 0)
-			(effects
-				(font
-					(size 1.27 1.27)
-				)
-				(justify left)
-			)
-		)
-		(property "Footprint" "MountingHole:MountingHole_5mm"
-			(at 208.28 41.91 0)
-			(effects
-				(font
-					(size 1.27 1.27)
-				)
-				(hide yes)
-			)
-		)
-		(property "Datasheet" "~"
-			(at 208.28 41.91 0)
-			(effects
-				(font
-					(size 1.27 1.27)
-				)
-				(hide yes)
-			)
-		)
-		(property "Description" "Mounting Hole without connection"
-			(at 208.28 41.91 0)
-			(effects
-				(font
-					(size 1.27 1.27)
-				)
-				(hide yes)
-			)
-		)
-		(instances
-			(project "LEMOAdaptorBoard4"
-				(path "/90a29a6b-0930-4b18-ad75-feedfe88ac78"
-					(reference "H3")
-					(unit 1)
-				)
-			)
-		)
-	)
-	(symbol
 		(lib_id "LEMO_Horizontal2:FPL.00.250.NTD")
 		(at 24.13 157.48 180)
@@
 				(path "/90a29a6b-0930-4b18-ad75-feedfe88ac78"
 					(reference "LEMO04")
+					(unit 1)
+				)
+			)
+		)
+	)
+	(symbol
+		(lib_id "Mechanical:MountingHole_Pad")
+		(at 205.74 54.61 0)
+		(unit 1)
+		(exclude_from_sim yes)
+		(in_bom no)
+		(on_board yes)
+		(dnp no)
+		(fields_autoplaced yes)
+		(property "Reference" "H3"
+			(at 208.28 52.0699 0)
+			(effects
+				(font
+					(size 1.27 1.27)
+				)
+				(justify left)
+			)
+		)
+		(property "Value" "MountingHole_Pad"
+			(at 208.28 54.6099 0)
+			(effects
+				(font
+					(size 1.27 1.27)
+				)
+				(justify left)
+			)
+		)
+		(property "Footprint" "MountingHole:MountingHole_5mm_Pad"
+			(at 205.74 54.61 0)
+			(effects
+				(font
+					(size 1.27 1.27)
+				)
+				(hide yes)
+			)
+		)
+		(property "Datasheet" "~"
+			(at 205.74 54.61 0)
+			(effects
+				(font
+					(size 1.27 1.27)
+				)
+				(hide yes)
+			)
+		)
+		(property "Description" "Mounting Hole with connection"
+			(at 205.74 54.61 0)
+			(effects
+				(font
+					(size 1.27 1.27)
+				)
+				(hide yes)
+			)
+		)
+		(pin "1"
+		)
+		(instances
+			(project "LEMOAdaptorBoard4"
+				(path "/90a29a6b-0930-4b18-ad75-feedfe88ac78"
+					(reference "H3")
 					(unit 1)
 				)
@@
 	)
 	(symbol
-		(lib_id "Mechanical:MountingHole")
-		(at 208.28 22.86 0)
+		(lib_id "Mechanical:MountingHole_Pad")
+		(at 205.74 66.04 0)
+		(unit 1)
+		(exclude_from_sim yes)
+		(in_bom no)
+		(on_board yes)
+		(dnp no)
+		(fields_autoplaced yes)
+		(property "Reference" "H4"
+			(at 208.28 63.4999 0)
+			(effects
+				(font
+					(size 1.27 1.27)
+				)
+				(justify left)
+			)
+		)
+		(property "Value" "MountingHole_Pad"
+			(at 208.28 66.0399 0)
+			(effects
+				(font
+					(size 1.27 1.27)
+				)
+				(justify left)
+			)
+		)
+		(property "Footprint" "MountingHole:MountingHole_5mm_Pad"
+			(at 205.74 66.04 0)
+			(effects
+				(font
+					(size 1.27 1.27)
+				)
+				(hide yes)
+			)
+		)
+		(property "Datasheet" "~"
+			(at 205.74 66.04 0)
+			(effects
+				(font
+					(size 1.27 1.27)
+				)
+				(hide yes)
+			)
+		)
+		(property "Description" "Mounting Hole with connection"
+			(at 205.74 66.04 0)
+			(effects
+				(font
+					(size 1.27 1.27)
+				)
+				(hide yes)
+			)
+		)
+		(pin "1"
+		)
+		(instances
+			(project "LEMOAdaptorBoard4"
+				(path "/90a29a6b-0930-4b18-ad75-feedfe88ac78"
+					(reference "H4")
+					(unit 1)
+				)
+			)
+		)
+	)
+	(symbol
+		(lib_id "Mechanical:MountingHole_Pad")
+		(at 205.74 30.48 0)
 		(unit 1)
 		(exclude_from_sim yes)
@@
 		(fields_autoplaced yes)
 		(property "Reference" "H1"
-			(at 210.82 21.5899 0)
+			(at 208.28 27.9399 0)
 			(effects
 				(font
@@
 			)
 		)
-		(property "Value" "MountingHole"
-			(at 210.82 24.1299 0)
+		(property "Value" "MountingHole_Pad"
+			(at 208.28 30.4799 0)
 			(effects
 				(font
@@
 			)
 		)
-		(property "Footprint" "MountingHole:MountingHole_5mm"
-			(at 208.28 22.86 0)
+		(property "Footprint" "MountingHole:MountingHole_5mm_Pad"
+			(at 205.74 30.48 0)
 			(effects
 				(font
@@
 		)
 		(property "Datasheet" "~"
-			(at 208.28 22.86 0)
-			(effects
-				(font
-					(size 1.27 1.27)
-				)
-				(hide yes)
-			)
-		)
-		(property "Description" "Mounting Hole without connection"
-			(at 208.28 22.86 0)
-			(effects
-				(font
-					(size 1.27 1.27)
-				)
-				(hide yes)
-			)
+			(at 205.74 30.48 0)
+			(effects
+				(font
+					(size 1.27 1.27)
+				)
+				(hide yes)
+			)
+		)
+		(property "Description" "Mounting Hole with connection"
+			(at 205.74 30.48 0)
+			(effects
+				(font
+					(size 1.27 1.27)
+				)
+				(hide yes)
+			)
+		)
+		(pin "1"
 		)
 		(instances
@@
 				(path "/90a29a6b-0930-4b18-ad75-feedfe88ac78"
 					(reference "H1")
+					(unit 1)
+				)
+			)
+		)
+	)
+	(symbol
+		(lib_id "Mechanical:MountingHole_Pad")
+		(at 205.74 43.18 0)
+		(unit 1)
+		(exclude_from_sim yes)
+		(in_bom no)
+		(on_board yes)
+		(dnp no)
+		(fields_autoplaced yes)
+		(property "Reference" "H2"
+			(at 208.28 40.6399 0)
+			(effects
+				(font
+					(size 1.27 1.27)
+				)
+				(justify left)
+			)
+		)
+		(property "Value" "MountingHole_Pad"
+			(at 208.28 43.1799 0)
+			(effects
+				(font
+					(size 1.27 1.27)
+				)
+				(justify left)
+			)
+		)
+		(property "Footprint" "MountingHole:MountingHole_5mm_Pad"
+			(at 205.74 43.18 0)
+			(effects
+				(font
+					(size 1.27 1.27)
+				)
+				(hide yes)
+			)
+		)
+		(property "Datasheet" "~"
+			(at 205.74 43.18 0)
+			(effects
+				(font
+					(size 1.27 1.27)
+				)
+				(hide yes)
+			)
+		)
+		(property "Description" "Mounting Hole with connection"
+			(at 205.74 43.18 0)
+			(effects
+				(font
+					(size 1.27 1.27)
+				)
+				(hide yes)
+			)
+		)
+		(pin "1"
+		)
+		(instances
+			(project "LEMOAdaptorBoard4"
+				(path "/90a29a6b-0930-4b18-ad75-feedfe88ac78"
+					(reference "H2")
 					(unit 1)
 				)
@@
 					(unit 1)
 				)
-			)
-		)
-	)
-	(symbol
-		(lib_id "Mechanical:MountingHole")
-		(at 208.28 33.02 0)
-		(unit 1)
-		(exclude_from_sim yes)
-		(in_bom no)
-		(on_board yes)
-		(dnp no)
-		(fields_autoplaced yes)
-		(property "Reference" "H2"
-			(at 210.82 31.7499 0)
-			(effects
-				(font
-					(size 1.27 1.27)
-				)
-				(justify left)
-			)
-		)
-		(property "Value" "MountingHole"
-			(at 210.82 34.2899 0)
-			(effects
-				(font
-					(size 1.27 1.27)
-				)
-				(justify left)
-			)
-		)
-		(property "Footprint" "MountingHole:MountingHole_5mm"
-			(at 208.28 33.02 0)
-			(effects
-				(font
-					(size 1.27 1.27)
-				)
-				(hide yes)
-			)
-		)
-		(property "Datasheet" "~"
-			(at 208.28 33.02 0)
-			(effects
-				(font
-					(size 1.27 1.27)
-				)
-				(hide yes)
-			)
-		)
-		(property "Description" "Mounting Hole without connection"
-			(at 208.28 33.02 0)
-			(effects
-				(font
-					(size 1.27 1.27)
-				)
-				(hide yes)
-			)
-		)
-		(instances
-			(project "LEMOAdaptorBoard4"
-				(path "/90a29a6b-0930-4b18-ad75-feedfe88ac78"
-					(reference "H2")
-					(unit 1)
-				)

Commit message: More update
Parts:
- added Power2: Conn_01x04, Connector:FanPinHeader_1x04_P2.54mm_Vertical, symbol Connector_Generic:Conn_01x04
Connections:
- net at FFC1.01 (Earth), FFC1.03 (Earth), FFC1.05 (Earth)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: now also Power2.4 (Pin_4)
- net at FFC1.07 (-2V5), FFC2.07 (-2V5), FFC3.07 (-2V5)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: now also Power2.3 (Pin_3)
- net at FFC1.08 (+2V5), FFC2.08 (+2V5), FFC3.08 (+2V5)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: now also Power2.2 (Pin_2)
- net at FFC1.09 (V_Bias), FFC2.09 (V_Bias), FFC3.09 (V_Bias)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: now also Power2.1 (Pin_1)
