File: SiPm_Design_2/SiPm_Design_2.kicad_pcb (KiCad board)
At the start: 2 copper layers, 125.8 x 12.5 mm, 20 parts, among them IC1 OPA354AIDBVTG4, IC2 AFBR-S4N44P014M, IC3 AFBR-S4N44P014M, IC4 AFBR-S4N44P014M, IC5 AFBR-S4N44P014M, J3 1-1734839-0

Commit message: add EM shield btm
Other:
- board text added: "EM shielding btm"
- board text added: "EM shielding top"
- board text added: "stiffener"
- board text removed: "EM shielding film"
- board text removed: "PI stiffener 0.225mm"
Changed lines of the file:
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@@
 		(49 "F.Fab" user)
 		(50 "User.1" user "Stiffener")
-		(51 "User.2" user "EM shilding film")
-		(52 "User.3" user)
+		(51 "User.2" user "EM shielding top")
+		(52 "User.3" user "EM shielding btm")
 		(53 "User.4" user)
 		(54 "User.5" user)
@@
 	(gr_rect
 		(start 184.138 103.204)
-		(end 247.888 112.204)
+		(end 245.729 112.204)
 		(stroke
 			(width 0.15)
@@
 		(layer "User.2")
 	)
+	(gr_rect
+		(start 184.138 103.204)
+		(end 245.729 112.204)
+		(stroke
+			(width 0.15)
+			(type default)
+		)
+		(fill solid)
+		(layer "User.3")
+	)
 	(gr_text "Vb"
 		(at 247.892 106.18 0)
@@
 		)
 	)
-	(gr_text "PI stiffener 0.225mm"
+	(gr_text "stiffener"
 		(at 164.388 100.204 0)
 		(layer "User.1")
@@
 		)
 	)
-	(gr_text "EM shielding film"
+	(gr_text "EM shielding top"
 		(at 196.138 100.454 0)
 		(layer "User.2")
 		(effects
 			(font
+				(size 1 1)
+				(thickness 0.15)
+			)
+			(justify left bottom)
+		)
+	)
+	(gr_text "EM shielding btm"
+		(at 210.173 100.465 0)
+		(layer "User.3")
+		(effects
+			(font

Commit message: Update stuff
Parts:
- C2: value 100n -> 10n
- R1: value 100 -> 1k
- R3: value 0 -> 10
- R4: value 50 -> 10
- R5: value 50 -> 0

Commit message: update first design
Parts:
- removed IC2, IC3, IC4, IC5: AFBR-S4N44P014M, S4N44P014M:AFBRS4N44P014M
- added U1: MICROFJ-30035-TSV-TR, MICROFJ_30035_TSV_TR:MicroFJ-300XX-TSV_ONS, F.Cu at (155.4, 108.9)
- IC1: footprint LIB_OPA354AIDBVTG4:SOT95P280X145-5N -> LMH6609MF_NOPB:SOT95P280X145-5N
Routing:
- net /anode: track 30.7 -> 5.81 mm
- net /Bias: track 43.1 -> 18.7 mm
Other:
- board size 125.8 x 12.5 mm -> 102.2 x 12.5 mm
