File: SiPm_Design_2/SiPm_Design_2.kicad_pcb (KiCad board)
At the start: 2 copper layers, 125.8 x 12.5 mm, 20 parts, among them IC1 OPA354AIDBVTG4, IC2 AFBR-S4N44P014M, IC3 AFBR-S4N44P014M, IC4 AFBR-S4N44P014M, IC5 AFBR-S4N44P014M, J3 1-1734839-0

Commit message: create new design3
Parts:
- removed IC4, IC5: AFBR-S4N44P014M, S4N44P014M:AFBRS4N44P014M
- added R7: 0, Resistor_SMD:R_0603_1608Metric_Pad0.98x0.95mm_HandSolder, F.Cu at (157.1, 108.9)
- IC3: value AFBR-S4N44P014M -> MICROFJ-30035-TSV-TR; footprint S4N44P014M:AFBRS4N44P014M -> J-30035:MICROFJ30035TSVTR
- R3, R4: value 10 -> 20
- R5: value 0 -> 50
- R6: value 50 -> 0
- moved R6 21.9 mm to (157.1, 107.2), turned to 0 degrees
- moved IC2 8.04 mm to (143.3, 107.7)
- moved IC3 4.16 mm to (149.1, 107.7)
Connections:
- net Earth renamed 0
- J3 pad 2: Net-(J3-Pad2) -> out
- J3 pad 4: Net-(J3-Pad2) -> out
- R2 pad 1: /anode -> /in
- R3 pad 2: /anode -> /in
- R5 pad 1: Net-(R5-Pad1) -> out
- R6 pad 1: Net-(J3-Pad2) -> /anode
- R6 pad 2: Net-(R5-Pad1) -> /in
Routing:
- net out: track 0.00 -> 152.5 mm, vias 0 -> 2
- net Net-(J3-Pad2): track 148.7 -> 0.00 mm, vias 1 -> 0
- net /anode: track 30.7 -> 13.5 mm, vias 0 -> 1
- net /Bias: track 43.1 -> 34.5 mm, vias 0 -> 7
- net /fastA: track 0.00 -> 8.03 mm
- net /in: track 0.00 -> 7.80 mm
- net Net-(R5-Pad1): track 4.05 -> 0.00 mm, vias 1 -> 0
- net 0: track 360.1 -> 358.0 mm, vias 17 -> 30
- net (no net): track 0.00 -> 2.02 mm, vias 0 -> 2
- added copper zone on B.Cu, net /Bias
- removed copper zone on F.Cu, net /Bias
Other:
- board size 125.8 x 12.5 mm -> 114.8 x 12.5 mm
- board text added: "2026 02 03 KK"
- board text removed: "2025 03 30 KK"
