File: SiPm_Design_2/SiPm_Design_2.kicad_sch (KiCad schematic)
At the start: 20 parts, among them IC1 OPA354AIDBVTG4, IC2 AFBR-S4N44P014M, IC3 AFBR-S4N44P014M, IC4 AFBR-S4N44P014M, IC5 AFBR-S4N44P014M, J3 1-1734839-0

Commit message: create new design3
Parts:
- removed IC3, IC4, IC5: AFBR-S4N44P014M, S4N44P014M:AFBRS4N44P014M, symbol AFBR-S4N44P014M:AFBR-S4N44P014M
- added IC3: MICROFJ-30035-TSV-TR, J-30035:MICROFJ30035TSVTR, symbol SamacSys_Parts:MICROFJ-30035-TSV-TR
- added R7: 0, Resistor_SMD:R_0603_1608Metric_Pad0.98x0.95mm_HandSolder, symbol Device:R
- added V1, V2: 2.5, symbol Simulation_SPICE:VDC
- added V4: VEXP, symbol Simulation_SPICE:VEXP
- added V5: VTRNOISE, symbol Simulation_SPICE:VTRNOISE
- IC1: footprint SOT95P280X145-5N -> LIB_OPA354AIDBVTG4:SOT95P280X145-5N
- R3, R4: value 10 -> 20
- R5: value 0 -> 50
- R6: value 50 -> 0
Connections:
- net +2V5: now also V1.1
- net -2V5: now also V2.2
- net Bias: now also IC3.A1 (CATHODE_1), IC3.A2 (NO_CONNECT_1), IC3.A3 (NO_CONNECT_2), IC3.C1 (NO_CONNECT_3), IC3.C2 (NO_CONNECT_4), IC3.C3 (CATHODE_2)
- net anode: now also R6.1, IC3.B1 (ANODE); no longer R2.1, R3.2
- net in: now reaches R6.2
- net in: now also R2.1, R3.2, R7.1, V4.1; no longer R5.1
- net out: now reaches J3.2, J3.4
- net out: now also R5.1; no longer R6.1
- net Earth renamed 0
- net 0: now also V1.2, V2.1, V4.2
- new net fastA: IC3.B3 (FAST_OUTPUT), R7.2
Other:
- note added: ".tran 10p 100n"
- moved on the sheet: C1, C2, C3, IC2, R1, R5, Rf1
